File: EEE3088F_Kicad/Sensor.kicad_sch (KiCad schematic)
At the start: 22 parts, among them IC1 AS5600-ASOT, U5 DRV5032FCDBZR, U6 MCP9700T-E/TT

Commit message: I have updated microcontoller and comments
Parts:
- renumbered R8 to R40, R8 to R41
Changed lines of the file:
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@@
   (symbol (lib_id "Device:R") (at 93.98 82.55 180) (unit 1)
     (in_bom yes) (on_board yes) (dnp no)
-    (property "Reference" "R8" (at 99.06 83.82 0)
+    (property "Reference" "R41" (at 99.06 83.82 0)
       (effects (font (size 1.27 1.27)) (justify left))
     )
@@
       (project "EEE3088F_Kicad"
         (path "/6f03c876-746d-4bbb-b455-2f8bb16ffc56/d0e1c216-fa44-4b75-912a-656721c3051d"
-          (reference "R8") (unit 1)
+          (reference "R41") (unit 1)
         )
       )
@@
   (symbol (lib_id "Device:R") (at 91.44 80.01 180) (unit 1)
     (in_bom yes) (on_board yes) (dnp no)
-    (property "Reference" "R8" (at 88.9 80.645 0)
+    (property "Reference" "R40" (at 88.9 80.645 0)
       (effects (font (size 1.27 1.27)) (justify left))
     )
@@
       (project "EEE3088F_Kicad"
         (path "/6f03c876-746d-4bbb-b455-2f8bb16ffc56/d0e1c216-fa44-4b75-912a-656721c3051d"
-          (reference "R8") (unit 1)
-        )
-      )
+          (reference "R40") (unit 1)
+        )
+      )

Commit message: I just added info to my title sectiion.
Parts:
- renumbered R41 to R8, R40 to R8
Other:
- company: UCT -> University of Cape Town
- moved on the sheet: C1, IC1, R1, R10, R2, R3, R4, R5, R6, R7, R8, R9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
